Commit message: Disfunctional xacro and launch file

File: homework2/twoarm.urdf.xacro (robot description, xacro)
@@ -1,2 +1,10 @@
+<?xml version = "1.0"?>
+<robot name="Part2" xmlns:xacro="http://www.ros.org/wiki/xacro">
+<xacro:property name="arm" value = "$(find homework2)/config/arm.yaml" />
+<xacro:property name="arm value = '$(load_yaml(arm))'/>
+<xacro:property name="L1" value="${arm['L1']}"/>
+<xacro:property name="L2" value="${arm['L2']}"/>
+<xacro:property name="R1" value="${arm['R1']}"/>
+<xacro:property name="R2" value="${arm['R2']}"/>
 <link name="base" >
   <visual>
@@ -22,5 +30,5 @@
    <origin xyz="0 0 0" rpy="0 0 0" />
    <geometry>
-     <cylinder radius="0.1" length="L1" />
+     <cylinder radius="0.1" length="${L1}" />
    </geometry>
      <material name="blue_mat">
@@ -31,5 +39,5 @@
      <origin xyz="0 0 0" rpy="0 0 0" />
    <geometry>
-     <cylinder radius="0.1" length="L1" />
+     <cylinder radius="0.1" length="${L1}" />
    </geometry>
    </collision>
@@ -43,5 +51,5 @@
   <origin xyz="0 0 0" rpy="0 0 0" />
    <geometry>
-     <cylinder radius="0.1" length="L2" />
+     <cylinder radius="0.1" length="${L2}" />
    </geometry>
      <material name="red_mat">
@@ -65,2 +73,3 @@
    </visual>
 </link>
+</robot>

Commit message: I have a horizontal pole

File: homework2/twoarm.urdf.xacro (robot description, xacro)
@@ -1,14 +1,9 @@
 <?xml version = "1.0"?>
 <robot name="Part2" xmlns:xacro="http://www.ros.org/wiki/xacro">
-<xacro:property name="arm" value = "$(find homework2)/config/arm.yaml" />
-<xacro:property name="arm value = '$(load_yaml(arm))'/>
-<xacro:property name="L1" value="${arm['L1']}"/>
-<xacro:property name="L2" value="${arm['L2']}"/>
-<xacro:property name="R1" value="${arm['R1']}"/>
-<xacro:property name="R2" value="${arm['R2']}"/>
 <link name="base" >
   <visual>
+    <origin xyz="0 0 0" rpy="0 1.571 0" />
     <geometry>
-      <sphere radius="0.1" />
+     <sphere radius="0.1" />
      </geometry>
      <material name="green_mat">
@@ -18,17 +13,18 @@
 </link>
 <joint name="base_joint" type="continuous">
-  <parent link="L1" />
-  <child link="L2" />
+  <parent link="base" />
+  <child link="L1" />
+  <origin xyz=".1 0 0" rpy="0 0 0" />
 </joint>
 <link name="L1">
    <inertial>
-     <origin xyz="0 0 0.5" rpy="0 0 0"/>
+     <origin xyz=".5 0 0" rpy="0 1.571 0"/>
      <mass value="1"/>
      <inertia ixx="100"  ixy="0"  ixz="0" iyy="100" iyz="0" izz="100" />
    </inertial>
   <visual>
-   <origin xyz="0 0 0" rpy="0 0 0" />
+   <origin xyz=".5 0 0" rpy="0 1.571 0" />
    <geometry>
-     <cylinder radius="0.1" length="${L1}" />
+     <cylinder radius="0.1" length="1" />
    </geometry>
      <material name="blue_mat">
@@ -37,7 +33,7 @@
   </visual>
   <collision>
-     <origin xyz="0 0 0" rpy="0 0 0" />
+     <origin xyz=".5 0 0" rpy="0 1.571 0" />
    <geometry>
-     <cylinder radius="0.1" length="${L1}" />
+     <cylinder radius="0.1" length="1" />
    </geometry>
    </collision>
@@ -46,10 +42,16 @@
   <parent link="L1" />
   <child link="L2" />
+  <origin xyz="1 0 0" rpy="0 0 0" />
 </joint>
 <link name="L2">
+   <inertial>
+     <origin xyz="1 0 0" rpy="0 1.571 0"/>
+     <mass value="1"/>
+     <inertia ixx="100"  ixy="0"  ixz="0" iyy="100" iyz="0" izz="100" />
+   </inertial>
   <visual>
-  <origin xyz="0 0 0" rpy="0 0 0" />
+  <origin xyz="1 0 0" rpy="0 1.571 0" />
    <geometry>
-     <cylinder radius="0.1" length="${L2}" />
+     <cylinder radius="0.1" length="2" />
    </geometry>
      <material name="red_mat">
@@ -57,17 +59,24 @@
      </material>
    </visual>
+  <collision>
+     <origin xyz="1 0 0" rpy="0 1.571 0" />
+   <geometry>
+     <cylinder radius="0.1" length="2" />
+   </geometry>
+   </collision>
 </link>
 <joint name="end_joint" type="fixed">
   <parent link="L2" />
   <child link="end" />
+  <origin xyz="2 0 0" rpy="0 0 0" />
 </joint>
 <link name="end">
   <visual>
-  <origin xyz="0 0 0" rpy="0 0 0" />
+  <origin xyz=".05 0 0" rpy="0 1.571 0" />
    <geometry>
      <cylinder radius="0.1" length=".1" />
    </geometry>
-     <material name="red_mat">
-         <color rgba="1 0 0 1" />
+     <material name="cyan_mat">
+         <color rgba="0 .5 .5 1" />
      </material>
    </visual>

Commit message: Joint calculations

File: homework2/twoarm.urdf.xacro (robot description, xacro)
@@ -1,5 +1,5 @@
 <?xml version = "1.0"?>
 <robot name="Part2" xmlns:xacro="http://www.ros.org/wiki/xacro">
-<link name="base" >
+<link name="base">
   <visual>
     <origin xyz="0 0 0" rpy="0 1.571 0" />
@@ -11,8 +11,15 @@
      </material>
    </visual>
+  <collision>
+    <origin xyz="0 0 0" rpy="0 1.571 0" />
+   <geometry>
+    <sphere radius="0.1" />
+   </geometry>
+   </collision>
 </link>
-<joint name="base_joint" type="continuous">
+<joint name="joint_1" type="continuous">
   <parent link="base" />
   <child link="L1" />
+  <axis xyz = "0 0 1" />
   <origin xyz=".1 0 0" rpy="0 0 0" />
 </joint>
@@ -39,7 +46,8 @@
    </collision>
 </link>
-<joint name="joint" type="continuous">
+<joint name="joint_2" type="continuous">
   <parent link="L1" />
   <child link="L2" />
+  <axis xyz = "0 0 1" />
   <origin xyz="1 0 0" rpy="0 0 0" />
 </joint>
@@ -69,4 +77,5 @@
   <parent link="L2" />
   <child link="end" />
+  <axis xyz = "0 0 1" />
   <origin xyz="2 0 0" rpy="0 0 0" />
 </joint>
@@ -75,8 +84,8 @@
   <origin xyz=".05 0 0" rpy="0 1.571 0" />
    <geometry>
-     <cylinder radius="0.1" length=".1" />
+     <cylinder radius=".1" length=".1" />
    </geometry>
-     <material name="cyan_mat">
-         <color rgba="0 .5 .5 1" />
+     <material name="invisible">
+         <color rgba="0 .5 .5 0" />
      </material>
    </visual>

Commit message: Added if statements to figure_eight.launch

File: homework2/twoarm.urdf.xacro (robot description, xacro)
@@ -6,9 +6,9 @@
     <geometry>
      <sphere radius="0.1" />
-     </geometry>
-     <material name="green_mat">
-         <color rgba="0 1 0 1" />
-     </material>
-   </visual>
+    </geometry>
+    <material name="green_mat">
+      <color rgba="0 1 0 1" />
+    </material>
+  </visual>
   <collision>
     <origin xyz="0 0 0" rpy="0 1.571 0" />
@@ -16,5 +16,5 @@
     <sphere radius="0.1" />
    </geometry>
-   </collision>
+  </collision>
 </link>
 <joint name="joint_1" type="continuous">
@@ -25,4 +25,5 @@
 </joint>
 <link name="L1">
+  <visual>
    <inertial>
      <origin xyz=".5 0 0" rpy="0 1.571 0"/>
@@ -30,5 +31,4 @@
      <inertia ixx="100"  ixy="0"  ixz="0" iyy="100" iyz="0" izz="100" />
    </inertial>
-  <visual>
    <origin xyz=".5 0 0" rpy="0 1.571 0" />
    <geometry>
@@ -44,5 +44,5 @@
      <cylinder radius="0.1" length="1" />
    </geometry>
-   </collision>
+  </collision>
 </link>
 <joint name="joint_2" type="continuous">
@@ -53,4 +53,5 @@
 </joint>
 <link name="L2">
+   <visual>
    <inertial>
      <origin xyz="1 0 0" rpy="0 1.571 0"/>
@@ -58,5 +59,4 @@
      <inertia ixx="100"  ixy="0"  ixz="0" iyy="100" iyz="0" izz="100" />
    </inertial>
-  <visual>
   <origin xyz="1 0 0" rpy="0 1.571 0" />
    <geometry>
@@ -66,11 +66,11 @@
          <color rgba="1 0 0 1" />
      </material>
-   </visual>
+  </visual>
   <collision>
      <origin xyz="1 0 0" rpy="0 1.571 0" />
-   <geometry>
+  <geometry>
      <cylinder radius="0.1" length="2" />
-   </geometry>
-   </collision>
+  </geometry>
+  </collision>
 </link>
 <joint name="end_joint" type="fixed">
@@ -86,8 +86,8 @@
      <cylinder radius=".1" length=".1" />
    </geometry>
-     <material name="invisible">
-         <color rgba="0 .5 .5 0" />
-     </material>
-   </visual>
+    <material name="invisible">
+      <color rgba="0 .5 .5 0" />
+    </material>
+  </visual>
 </link>
 </robot>

Commit message: Added parameters to xacro files, checking for substitution errors

File: homework2/twoarm.urdf.xacro (robot description, xacro)
@@ -1,4 +1,10 @@
 <?xml version = "1.0"?>
 <robot name="Part2" xmlns:xacro="http://www.ros.org/wiki/xacro">
+<xacro:property name="armyaml" value = "$(find homework2)/config/arm.yaml" />
+<xacro:property name="arm" value = '${load_yaml (armyaml)}'/>
+<xacro:property name="L1" value="${arm['L1']}"/>
+<xacro:property name="L2" value="${arm['L2']}"/>
+<xacro:property name="R1" value="${arm['R1']}"/>
+<xacro:property name="R2" value="${arm['R2']}"/>
 <link name="base">
   <visual>
@@ -33,5 +39,5 @@
    <origin xyz=".5 0 0" rpy="0 1.571 0" />
    <geometry>
-     <cylinder radius="0.1" length="1" />
+     <cylinder radius="${R1}" length="${L1}" />
    </geometry>
      <material name="blue_mat">
@@ -42,5 +48,5 @@
      <origin xyz=".5 0 0" rpy="0 1.571 0" />
    <geometry>
-     <cylinder radius="0.1" length="1" />
+     <cylinder radius="${R1}" length="${L1}" />
    </geometry>
   </collision>

Commit message: Subbed in parameters

File: homework2/twoarm.urdf.xacro (robot description, xacro)
@@ -37,5 +37,5 @@
      <inertia ixx="100"  ixy="0"  ixz="0" iyy="100" iyz="0" izz="100" />
    </inertial>
-   <origin xyz=".5 0 0" rpy="0 1.571 0" />
+   <origin xyz="${L1/2} 0 0" rpy="0 1.571 0" />
    <geometry>
      <cylinder radius="${R1}" length="${L1}" />
@@ -46,5 +46,5 @@
   </visual>
   <collision>
-     <origin xyz=".5 0 0" rpy="0 1.571 0" />
+     <origin xyz="${L1/2} 0 0" rpy="0 1.571 0" />
    <geometry>
      <cylinder radius="${R1}" length="${L1}" />
@@ -61,5 +61,5 @@
    <visual>
    <inertial>
-     <origin xyz="1 0 0" rpy="0 1.571 0"/>
+     <origin xyz="${L2/2} 0 0" rpy="0 1.571 0"/>
      <mass value="1"/>
      <inertia ixx="100"  ixy="0"  ixz="0" iyy="100" iyz="0" izz="100" />
@@ -67,5 +67,5 @@
   <origin xyz="1 0 0" rpy="0 1.571 0" />
    <geometry>
-     <cylinder radius="0.1" length="2" />
+     <cylinder radius="${R2}" length="${L2}" />
    </geometry>
      <material name="red_mat">
@@ -76,5 +76,5 @@
      <origin xyz="1 0 0" rpy="0 1.571 0" />
   <geometry>
-     <cylinder radius="0.1" length="2" />
+     <cylinder radius="${R2}" length="${L2}" />
   </geometry>
   </collision>
@@ -84,5 +84,5 @@
   <child link="end" />
   <axis xyz = "0 0 1" />
-  <origin xyz="2 0 0" rpy="0 0 0" />
+  <origin xyz="${L2} 0 0" rpy="0 0 0" />
 </joint>
 <link name="end">

Commit message: Integrated parameters

File: homework2/twoarm.urdf.xacro (robot description, xacro)
@@ -56,5 +56,5 @@
   <child link="L2" />
   <axis xyz = "0 0 1" />
-  <origin xyz="1 0 0" rpy="0 0 0" />
+  <origin xyz="${L1} 0 0" rpy="0 0 0" />
 </joint>
 <link name="L2">
@@ -65,5 +65,5 @@
      <inertia ixx="100"  ixy="0"  ixz="0" iyy="100" iyz="0" izz="100" />
    </inertial>
-  <origin xyz="1 0 0" rpy="0 1.571 0" />
+  <origin xyz="${L2/2} 0 0" rpy="0 1.571 0" />
    <geometry>
      <cylinder radius="${R2}" length="${L2}" />
@@ -74,5 +74,5 @@
   </visual>
   <collision>
-     <origin xyz="1 0 0" rpy="0 1.571 0" />
+     <origin xyz="${L2/2} 0 0" rpy="0 1.571 0" />
   <geometry>
      <cylinder radius="${R2}" length="${L2}" />

Commit message: Implementing period parameter in arm_marker

File: homework2/twoarm.urdf.xacro (robot description, xacro)
@@ -33,5 +33,5 @@
   <visual>
    <inertial>
-     <origin xyz=".5 0 0" rpy="0 1.571 0"/>
+     <origin xyz="${L1/2} 0 0" rpy="0 1.571 0"/>
      <mass value="1"/>
      <inertia ixx="100"  ixy="0"  ixz="0" iyy="100" iyz="0" izz="100" />
